File: hardware/HeadphoneBoard/HeadphoneJack.sch (KiCad schematic (older format))
At the start: 8 parts, among them J1 8P8C

Commit message: 3.5mm Control, 3rd Button update, and new 28 pins
Created a new Headphone Jack board to control cars with more standardized control systems. Added a third analog button to the Joystick board to allow for 3 button control. Added a configuration jumper to the 28 pin control boards to allow 3rd button control toggle. Created a new control board that integrates the buck converter into the board.
Parts:
- added S3: Switch1, Useful Modifications:Jack_3.5mm_PJ320A_Horizontal_Short, symbol Connector:AudioJack4
- added S4: Switch2, Useful Modifications:Jack_3.5mm_PJ320A_Horizontal_Short, symbol Connector:AudioJack4
- J1: footprint Connector_RJ:RJ45_Amphenol_54602-x08_Horizontal -> Useful Modifications:RJ45_x08_Horizontal_tabs
- VR1: value JoyX -> Left; footprint Connector_PinHeader_2.54mm:PinHeader_1x03_P2.54mm_Vertical -> Useful Modifications:Jack_3.5mm_PJ320A_Horizontal_Short; symbol Connector:Conn_01x03_Male -> Connector:AudioJack4
- VR2: value JoyY -> Drive; footprint Connector_PinHeader_2.54mm:PinHeader_1x03_P2.54mm_Vertical -> Useful Modifications:Jack_3.5mm_PJ320A_Horizontal_Short; symbol Connector:Conn_01x03_Male -> Connector:AudioJack4
- VR3: value Optional Input -> Right; footprint Connector_PinHeader_2.54mm:PinHeader_1x03_P2.54mm_Vertical -> Useful Modifications:Jack_3.5mm_PJ320A_Horizontal_Short; symbol Connector:Conn_01x03_Male -> Connector:AudioJack4
Connections:
- wire segments 11 -> 19
- no-connect marks 0 -> 10
Other:
- note removed: "G S 3"
Changed lines of the file:
@@
 F 0 "J1" V 5211 3330 50  0000 L CNN
 F 1 "8P8C" V 5302 3330 50  0000 L CNN
-F 2 "Connector_RJ:RJ45_Amphenol_54602-x08_Horizontal" V 5200 2825 50  0001 C CNN
+F 2 "Useful Modifications:RJ45_x08_Horizontal_tabs" V 5200 2825 50  0001 C CNN
 F 3 "~" V 5200 2825 50  0001 C CNN
 	1    5200 2800
@@
 $EndComp
 $Comp
-L Connector:Conn_01x03_Male VR1
+L Connector:AudioJack4 VR1
 U 1 1 5D5C41B7
-P 5400 4050
-F 0 "VR1" V 5554 3862 50  0000 R CNN
-F 1 "JoyX" V 5463 3862 50  0000 R CNN
-F 2 "Connector_PinHeader_2.54mm:PinHeader_1x03_P2.54mm_Vertical" H 5400 4050 50  0001 C CNN
-F 3 "~" H 5400 4050 50  0001 C CNN
-	1    5400 4050
-	0    -1   -1   0
-$EndComp
-$Comp
-L Connector:Conn_01x03_Male VR2
+P 5200 4800
+F 0 "VR1" V 4900 4950 50  0000 R CNN
+F 1 "Left" V 4800 4950 50  0000 R CNN
+F 2 "Useful Modifications:Jack_3.5mm_PJ320A_Horizontal_Short" H 5200 4800 50  0001 C CNN
+F 3 "~" H 5200 4800 50  0001 C CNN
+	1    5200 4800
+	0    -1   -1   0
+$EndComp
+$Comp
+L Connector:AudioJack4 VR2
 U 1 1 5D5C5C5F
-P 5800 4550
-F 0 "VR2" V 5954 4362 50  0000 R CNN
-F 1 "JoyY" V 5863 4362 50  0000 R CNN
-F 2 "Connector_PinHeader_2.54mm:PinHeader_1x03_P2.54mm_Vertical" H 5800 4550 50  0001 C CNN
-F 3 "~" H 5800 4550 50  0001 C CNN
-	1    5800 4550
+P 5800 4800
+F 0 "VR2" V 5500 4950 50  0000 R CNN
+F 1 "Drive" V 5400 4950 50  0000 R CNN
+F 2 "Useful Modifications:Jack_3.5mm_PJ320A_Horizontal_Short" H 5800 4800 50  0001 C CNN
+F 3 "~" H 5800 4800 50  0001 C CNN
+	1    5800 4800
 	0    -1   -1   0
 $EndComp
@@
 Text Notes 5050 4400 0    59   ~ 0
 G S
-Text Notes 5650 4650 0    59   ~ 0
-G S 3
 $Comp
 L power:GND #PWR01
@@
 L power:GND #PWR09
 U 1 1 5D6B0365
-P 5300 3850
-F 0 "#PWR09" H 5300 3600 50  0001 C CNN
-F 1 "GND" H 5305 3677 50  0000 C CNN
-F 2 "" H 5300 3850 50  0001 C CNN
-F 3 "" H 5300 3850 50  0001 C CNN
-	1    5300 3850
+P 5100 4600
+F 0 "#PWR09" H 5100 4350 50  0001 C CNN
+F 1 "GND" H 5105 4427 50  0000 C CNN
+F 2 "" H 5100 4600 50  0001 C CNN
+F 3 "" H 5100 4600 50  0001 C CNN
+	1    5100 4600
 	-1   0    0    1
 $EndComp
@@
 L power:GND #PWR012
 U 1 1 5D6B136B
-P 5700 4350
-F 0 "#PWR012" H 5700 4100 50  0001 C CNN
-F 1 "GND" H 5705 4177 50  0000 C CNN
-F 2 "" H 5700 4350 50  0001 C CNN
-F 3 "" H 5700 4350 50  0001 C CNN
-	1    5700 4350
-	-1   0    0    1
-$EndComp
-$Comp
-L power:+3.3V #PWR011
-U 1 1 5D6B1B5E
-P 5500 3850
-F 0 "#PWR011" H 5500 3700 50  0001 C CNN
-F 1 "+3.3V" H 5515 4023 50  0000 C CNN
-F 2 "" H 5500 3850 50  0001 C CNN
-F 3 "" H 5500 3850 50  0001 C CNN
-	1    5500 3850
-	1    0    0    -1
-$EndComp
-$Comp
-L power:+3.3V #PWR013
-U 1 1 5D6B3F0F
-P 5900 4350
-F 0 "#PWR013" H 5900 4200 50  0001 C CNN
-F 1 "+3.3V" H 5915 4523 50  0000 C CNN
-F 2 "" H 5900 4350 50  0001 C CNN
-F 3 "" H 5900 4350 50  0001 C CNN
-	1    5900 4350
-	1    0    0    -1
+P 5700 4600
+F 0 "#PWR012" H 5700 4350 50  0001 C CNN
+F 1 "GND" H 5705 4427 50  0000 C CNN
+F 2 "" H 5700 4600 50  0001 C CNN
+F 3 "" H 5700 4600 50  0001 C CNN
+	1    5700 4600
+	-1   0    0    1
 $EndComp
 $Comp
@@
 $EndComp
 Wire Wire Line
-	5400 3650 5400 3850
-Wire Wire Line
-	5100 3200 5100 3650
-Wire Wire Line
-	5200 3200 5200 4100
-Wire Wire Line
 	5300 3200 5300 3550
 Wire Wire Line
@@
 Wire Wire Line
 	5400 3200 5400 3500
-Wire Wire Line
-	5400 3500 5800 3700
-Wire Wire Line
-	5800 3700 5800 4350
-$Comp
-L Connector:Conn_01x03_Male VR3
+$Comp
+L Connector:AudioJack4 VR3
 U 1 1 5EE05BA7
-P 6450 4550
-F 0 "VR3" V 6604 4362 50  0000 R CNN
-F 1 "Optional Input" V 6513 4362 50  0000 R CNN
-F 2 "Connector_PinHeader_2.54mm:PinHeader_1x03_P2.54mm_Vertical" H 6450 4550 50  0001 C CNN
-F 3 "~" H 6450 4550 50  0001 C CNN
-	1    6450 4550
+P 6450 4800
+F 0 "VR3" V 6150 4950 50  0000 R CNN
+F 1 "Right" V 6050 4950 50  0000 R CNN
+F 2 "Useful Modifications:Jack_3.5mm_PJ320A_Horizontal_Short" H 6450 4800 50  0001 C CNN
+F 3 "~" H 6450 4800 50  0001 C CNN
+	1    6450 4800
 	0    -1   -1   0
 $EndComp
@@
 L power:GND #PWR014
 U 1 1 5EE0785D
-P 6350 4350
-F 0 "#PWR014" H 6350 4100 50  0001 C CNN
-F 1 "GND" H 6355 4177 50  0000 C CNN
-F 2 "" H 6350 4350 50  0001 C CNN
-F 3 "" H 6350 4350 50  0001 C CNN
-	1    6350 4350
-	-1   0    0    1
-$EndComp
-$Comp
-L power:+3.3V #PWR015
-U 1 1 5EE0915C
-P 6550 4350
-F 0 "#PWR015" H 6550 4200 50  0001 C CNN
-F 1 "+3.3V" H 6565 4523 50  0000 C CNN
-F 2 "" H 6550 4350 50  0001 C CNN
-F 3 "" H 6550 4350 50  0001 C CNN
-	1    6550 4350
-	1    0    0    -1
-$EndComp
-Text Notes 6300 4650 0    59   ~ 0
-G S 3
+P 6350 4600
+F 0 "#PWR014" H 6350 4350 50  0001 C CNN
+F 1 "GND" H 6355 4427 50  0000 C CNN
+F 2 "" H 6350 4600 50  0001 C CNN
+F 3 "" H 6350 4600 50  0001 C CNN
+	1    6350 4600
+	-1   0    0    1
+$EndComp
 Wire Wire Line
 	5600 3200 5600 3450
 Wire Wire Line
-	5600 3450 6450 3900
-Wire Wire Line
-	6450 3900 6450 4350
+	5600 3450 6650 4000
+NoConn ~ 6550 4600
+NoConn ~ 6450 4600
+Wire Wire Line
+	5400 3500 6000 3800
+NoConn ~ 5900 4600
+NoConn ~ 5800 4600
+Wire Wire Line
+	5400 3650 5400 4600
+Wire Wire Line
+	6650 4000 6650 4600
+Wire Wire Line
+	6000 3800 6000 4600
+NoConn ~ 5200 4600
+NoConn ~ 5300 4600
+$Comp
+L Connector:AudioJack4 S4
+U 1 1 5EE20781
+P 4400 4800
+F 0 "S4" V 4100 4950 50  0000 R CNN
+F 1 "Switch2" V 4000 4950 50  0000 R CNN
+F 2 "Useful Modifications:Jack_3.5mm_PJ320A_Horizontal_Short" H 4400 4800 50  0001 C CNN
+F 3 "~" H 4400 4800 50  0001 C CNN
+	1    4400 4800
+	0    -1   -1   0
+$EndComp
+$Comp
+L Connector:AudioJack4 S3
+U 1 1 5EE21518
+P 3600 4800
+F 0 "S3" V 3300 4950 50  0000 R CNN
+F 1 "Switch1" V 3200 4950 50  0000 R CNN
+F 2 "Useful Modifications:Jack_3.5mm_PJ320A_Horizontal_Short" H 3600 4800 50  0001 C CNN
+F 3 "~" H 3600 4800 50  0001 C CNN
+	1    3600 4800
+	0    -1   -1   0
+$EndComp
+$Comp
+L power:GND #PWR011
+U 1 1 5EE243B2
+P 3500 4600
+F 0 "#PWR011" H 3500 4350 50  0001 C CNN
+F 1 "GND" H 3500 4450 50  0000 C CNN
+F 2 "" H 3500 4600 50  0001 C CNN
+F 3 "" H 3500 4600 50  0001 C CNN
+	1    3500 4600
+	-1   0    0    1
+$EndComp
+$Comp
+L power:GND #PWR013
+U 1 1 5EE24899
+P 4300 4600
+F 0 "#PWR013" H 4300 4350 50  0001 C CNN
+F 1 "GND" H 4300 4450 50  0000 C CNN
+F 2 "" H 4300 4600 50  0001 C CNN
+F 3 "" H 4300 4600 50  0001 C CNN
+	1    4300 4600
+	-1   0    0    1
+$EndComp
+Wire Wire Line
+	5100 3200 5100 3350
+Wire Wire Line
+	5200 3800 4600 4200
+Wire Wire Line
+	4600 4200 4600 4600
+Wire Wire Line
+	5200 3200 5200 3800
+Wire Wire Line
+	5200 3800 5200 4100
+Connection ~ 5200 3800
+Wire Wire Line
+	5100 3350 4600 3700
+Wire Wire Line
+	4600 3700 4600 3900
+Wire Wire Line
+	4600 3900 3800 4350
+Wire Wire Line
+	3800 4350 3800 4600
+Connection ~ 5100 3350
+Wire Wire Line
+	5100 3350 5100 3650
+NoConn ~ 4500 4600
+NoConn ~ 4400 4600
+NoConn ~ 3700 4600
+NoConn ~ 3600 4600
 $EndSCHEMATC
