File: hardware/VS1000SimpleBreakout/VS1000SimpleBreakout.sch (KiCad schematic (older format))
At the start: 42 parts, among them J1 Conn_01x14, J2 AudioJack4, J3 USB_B_Micro, J4 Conn_01x14, U1 MX25R3235FM2xx0, U2 VS1000, Y1 Resonator

Commit message: vs1000 breakout PCB updates
Parts:
- Y1: DigiKey (none) -> https://www.digikey.com/en/products/detail/AWSCR-12.00CELA-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
Changed lines of the file:
@@
 F 2 "Project:Resonator" H 7795 5070 50  0001 C CNN
 F 3 "~" H 7795 5070 50  0001 C CNN
+F 4 "https://www.digikey.com/en/products/detail/AWSCR-12.00CELA-C33-T3/535-15066-1-ND/10232593?itemSeq=340296092" V 7820 5070 50  0001 C CNN "DigiKey"
 	1    7820 5070
 	0    -1   -1   0
