File: hardware/HallSensorSMD_9_Pos/HallSensorSMD_9_Pos.kicad_pcb (KiCad board)
At the start: 2 copper layers, 46.9 x 21.5 mm, 13 parts, among them J1 Power/Signal, U1 ATtiny814-SS, U10 Hall 9, U2 Hall 1, U3 Hall 2, U4 Hall 3, U5 Hall 4, U6 Hall 5, U7 Hall 6, U8 Hall 7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

Commit message: updating Hall Sensor 9 Position pin assignments
Parts:
- U10: value Hall 9 -> Hall 8
- U9: value Hall 8 -> Hall 9
Connections:
- J1 pad 1: Net-(J1-Pad1) -> GND
- J1 pad 2: GND -> Net-(J1-Pad2)
- U1 pad 7: Net-(U1-Pad7) -> Net-(J1-Pad2)
- U1 pad 9: Net-(J1-Pad1) -> Net-(U1-Pad9)
- U10 pad 2: Net-(U1-Pad7) -> Net-(U1-Pad9)
- U9 pad 2: Net-(U1-Pad6) -> Net-(U1-Pad8)
Routing:
- net Net-(U1-Pad9): track 0.00 -> 35.9 mm, vias 0 -> 1
- net Net-(U1-Pad8): track 0.00 -> 29.1 mm, vias 0 -> 1
- net Net-(U1-Pad7): track 23.9 -> 0.00 mm, vias 1 -> 0
- net Net-(J1-Pad2): track 0.00 -> 22.7 mm, vias 0 -> 2
- net Net-(U1-Pad6): track 20.8 -> 0.00 mm, vias 1 -> 0
- net Net-(J1-Pad1): track 13.4 -> 0.00 mm
- net +3V3: track 47.9 -> 44.7 mm, vias 0 -> 1
- net Net-(J1-Pad4): vias 0 -> 1

Commit message: gerbers for HallSensor and InputBoard PCBs, updates to HallSensor PCBs
Connections:
- J1 pad 1: GND -> Net-(J1-Pad1)
- J1 pad 2: Net-(J1-Pad2) -> GND
- U1 pad 7: Net-(J1-Pad2) -> Net-(J1-Pad1)
Routing:
- net Net-(J1-Pad1): track 0.00 -> 27.9 mm, vias 0 -> 2
- net Net-(J1-Pad2): track 22.7 -> 0.00 mm, vias 2 -> 0
Other:
- board text added: "9 Pos Hall Sensor V2"
- board text removed: "9 Pos Hall Sensor V1"
- board text removed: "RX"
- board text removed: "TX"
Changed lines of the file:
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@@
   (general
     (thickness 1.6)
-    (drawings 17)
-    (tracks 195)
+    (drawings 19)
+    (tracks 202)
     (zones 0)
     (modules 13)
@@
   (net 12 "Net-(U1-Pad6)")
   (net 13 "Net-(U1-Pad9)")
-  (net 14 "Net-(J1-Pad2)")
+  (net 14 "Net-(J1-Pad1)")
   (net_class Default "This is the default net class."
     (clearance 0.2)
@@
     (add_net +3V3)
     (add_net GND)
-    (add_net "Net-(J1-Pad2)")
+    (add_net "Net-(J1-Pad1)")
     (add_net "Net-(J1-Pad4)")
     (add_net "Net-(U1-Pad11)")
@@
     )
     (pad 1 thru_hole rect (at 0 0 90) (size 1.7 1.7) (drill 1) (layers *.Cu *.Mask)
-      (net 1 GND))
+      (net 14 "Net-(J1-Pad1)"))
     (pad 2 thru_hole oval (at 0 2.54 90) (size 1.7 1.7) (drill 1) (layers *.Cu *.Mask)
-      (net 14 "Net-(J1-Pad2)"))
+      (net 1 GND))
     (pad 3 thru_hole oval (at 0 5.08 90) (size 1.7 1.7) (drill 1) (layers *.Cu *.Mask)
       (net 5 +3V3))
@@
       (net 12 "Net-(U1-Pad6)"))
     (pad 7 smd roundrect (at -2.475 -3.81 135) (size 1.95 0.6) (layers B.Cu B.Paste B.Mask) (roundrect_rratio 0.25)
-      (net 14 "Net-(J1-Pad2)"))
+      (net 14 "Net-(J1-Pad1)"))
     (pad 8 smd roundrect (at 2.475 -3.81 135) (size 1.95 0.6) (layers B.Cu B.Paste B.Mask) (roundrect_rratio 0.25)
       (net 10 "Net-(U1-Pad8)"))
@@
     (tags SOT-23)
     (attr smd)
-    (fp_text reference U6 (at 0.318728 -2.3069) (layer F.SilkS)
+    (fp_text reference U6 (at 1.74 -0.965) (layer F.SilkS)
       (effects (font (size 0.762 0.762) (thickness 0.1397)))
     )
@@
     (tags SOT-23)
     (attr smd)
-    (fp_text reference U7 (at -2.438489 -0.266628 166) (layer F.SilkS)
+    (fp_text reference U7 (at 1.636135 -2.283651 166) (layer F.SilkS)
       (effects (font (size 0.762 0.762) (thickness 0.1397)))
     )
@@
     (tags SOT-23)
     (attr smd)
-    (fp_text reference U8 (at -2.459231 -0.620345 152) (layer F.SilkS)
+    (fp_text reference U8 (at 1.519378 -2.297197 152) (layer F.SilkS)
       (effects (font (size 0.762 0.762) (thickness 0.1397)))
     )
@@
     )
   )
+  (gr_text RST (at 133.6607 50.0765) (layer B.SilkS)
+    (effects (font (size 0.762 0.762) (thickness 0.1397)) (justify mirror))
+  )
+  (gr_text 3.3V (at 130.975 50.125) (layer B.SilkS)
+    (effects (font (size 0.6858 0.6858) (thickness 0.13335)) (justify mirror))
+  )
+  (gr_text GND (at 128.4 50.1) (layer B.SilkS)
+    (effects (font (size 0.6604 0.6604) (thickness 0.13335)) (justify mirror))
+  )
+  (gr_text PWM (at 125.8066 50.087) (layer B.SilkS)
+    (effects (font (size 0.762 0.762) (thickness 0.1397)) (justify mirror))
+  )
   (gr_arc (start 130 70.25) (end 153.499999 65.250001) (angle -154.8159682) (layer Edge.Cuts) (width 0.05))
   (gr_line (start 118.303073 67.512421) (end 106.606142 64.774841) (layer Edge.Cuts) (width 0.05))
@@
   (gr_line (start 119.95 63.1) (end 110.25 56.75) (layer F.SilkS) (width 0.12))
   (gr_line (start 139.9 63.2) (end 149.75 56.75) (layer F.SilkS) (width 0.12))
-  (gr_text "9 Pos Hall Sensor V1" (at 129.5654 56.896) (layer F.SilkS)
+  (gr_text "9 Pos Hall Sensor V2" (at 129.5654 56.896) (layer F.SilkS)
     (effects (font (size 0.762 0.762) (thickness 0.1397)))
   )
-  (gr_text RX (at 138.45 51.55 -35) (layer F.SilkS)
-    (effects (font (size 0.6858 0.6858) (thickness 0.13335)))
-  )
-  (gr_text TX (at 140.71 53.11 -35) (layer F.SilkS)
-    (effects (font (size 0.6858 0.6858) (thickness 0.13335)))
-  )
-  (gr_text GND (at 142.83 54.6 -35) (layer F.SilkS)
+  (gr_text GND (at 128.35 49.95) (layer F.SilkS)
     (effects (font (size 0.6604 0.6604) (thickness 0.13335)))
   )
-  (gr_text 3.3V (at 145.14 56.05 -35) (layer F.SilkS)
+  (gr_text 3.3V (at 131.1 49.875) (layer F.SilkS)
     (effects (font (size 0.6858 0.6858) (thickness 0.13335)))
   )
@@
   (segment (start 142.316537 56.687765) (end 144.298576 58.669804) (width 0.25) (layer F.Cu) (net 1))
   (segment (start 141.713145 56.369131) (end 142.031779 56.687765) (width 0.25) (layer F.Cu) (net 1))
-  (segment (start 126.681084 50.597634) (end 127.063711 50.980261) (width 0.25) (layer B.Cu) (net 1))
-  (segment (start 125.8189 48.25) (end 125.8189 49.73545) (width 0.25) (layer B.Cu) (net 1))
   (via (at 127.063711 50.980261) (size 0.8) (drill 0.4) (layers F.Cu B.Cu) (net 1))
-  (segment (start 125.8189 49.73545) (end 127.063711 50.980261) (width 0.25) (layer B.Cu) (net 1))
-  (segment (start 121.454288 50.597634) (end 126.681084 50.597634) (width 0.25) (layer B.Cu) (net 1))
   (segment (start 127.120296 51.036846) (end 127.063711 50.980261) (width 0.25) (layer F.Cu) (net 1))
   (segment (start 127.120296 52.208078) (end 127.120296 51.036846) (width 0.25) (layer F.Cu) (net 1))
+  (segment (start 126.681084 50.597634) (end 127.063711 50.980261) (width 0.25) (layer B.Cu) (net 1))
+  (segment (start 121.454288 50.597634) (end 126.681084 50.597634) (width 0.25) (layer B.Cu) (net 1))
+  (segment (start 128.3589 49.685072) (end 127.063711 50.980261) (width 0.25) (layer B.Cu) (net 1))
+  (segment (start 128.3589 48.25) (end 128.3589 49.685072) (width 0.25) (layer B.Cu) (net 1))
   (segment (start 116.600118 59.63165) (end 118.100034 58.131734) (width 0.25) (layer F.Cu) (net 2))
   (via (at 118.100034 57.596517) (size 0.8) (drill 0.4) (layers F.Cu B.Cu) (net 2))
@@
   (segment (start 120.788427 49.425001) (end 122.674999 49.425001) (width 0.25) (layer B.Cu) (net 11))
   (segment (start 122.674999 49.425001) (end 122.675 49.425) (width 0.25) (layer B.Cu) (net 11))
+  (segment (start 132.263899 47.074999) (end 132.588901 47.400001) (width 0.25) (layer F.Cu) (net 11))
   (segment (start 132.588901 47.400001) (end 133.4389 48.25) (width 0.25) (layer F.Cu) (net 11))
-  (segment (start 132.263899 47.074999) (end 132.588901 47.400001) (width 0.25) (layer F.Cu) (net 11))
-  (segment (start 127.794899 47.074999) (end 132.263899 47.074999) (width 0.25) (layer F.Cu) (net 11))
-  (segment (start 127.183899 47.685999) (end 127.794899 47.074999) (width 0.25) (layer F.Cu) (net 11))
-  (segment (start 127.183899 49.170003) (end 127.183899 47.685999) (width 0.25) (layer F.Cu) (net 11))
-  (segment (start 126.928902 49.425) (end 127.183899 49.170003) (width 0.25) (layer F.Cu) (net 11))
-  (segment (start 122.675 49.425) (end 126.928902 49.425) (width 0.25) (layer F.Cu) (net 11))
+  (segment (start 123.240685 49.425) (end 123.365685 49.55) (width 0.25) (layer F.Cu) (net 11))
+  (segment (start 122.675 49.425) (end 123.240685 49.425) (width 0.25) (layer F.Cu) (net 11))
+  (segment (start 129.723899 47.685999) (end 130.334899 47.074999) (width 0.25) (layer F.Cu) (net 11))
+  (segment (start 129.723899 49.076101) (end 129.723899 47.685999) (width 0.25) (layer F.Cu) (net 11))
+  (segment (start 129.25 49.55) (end 129.723899 49.076101) (width 0.25) (layer F.Cu) (net 11))
+  (segment (start 130.334899 47.074999) (end 132.263899 47.074999) (width 0.25) (layer F.Cu) (net 11))
+  (segment (start 123.365685 49.55) (end 129.25 49.55) (width 0.25) (layer F.Cu) (net 11))
   (via (at 137.175 57.65) (size 0.8) (drill 0.4) (layers F.Cu B.Cu) (net 13))
   (segment (start 141.897483 57.65) (end 142.373229 58.125746) (width 0.25) (layer F.Cu) (net 13))
@@
   (via (at 131.125 55.575) (size 0.8) (drill 0.4) (layers F.Cu B.Cu) (net 14))
   (segment (start 131.125 55.575) (end 132.125 54.575) (width 0.25) (layer B.Cu) (net 14))
-  (segment (start 132.125 52.0161) (end 128.3589 48.25) (width 0.25) (layer B.Cu) (net 14))
   (segment (start 132.125 54.575) (end 132.125 52.0161) (width 0.25) (layer B.Cu) (net 14))
+  (segment (start 125.8189 47.15) (end 125.8189 48.25) (width 0.25) (layer B.Cu) (net 14))
+  (segment (start 125.893901 47.074999) (end 125.8189 47.15) (width 0.25) (layer B.Cu) (net 14))
+  (segment (start 128.922901 47.074999) (end 125.893901 47.074999) (width 0.25) (layer B.Cu) (net 14))
+  (segment (start 129.723899 47.875997) (end 128.922901 47.074999) (width 0.25) (layer B.Cu) (net 14))
+  (segment (start 129.723899 49.614999) (end 129.723899 47.875997) (width 0.25) (layer B.Cu) (net 14))
+  (segment (start 132.125 52.0161) (end 129.723899 49.614999) (width 0.25) (layer B.Cu) (net 14))
 )
