File: hardware/ControlBoardnRF_22PinSound_PowerAmp/MAX9744.sch (KiCad schematic (older format))
At the start: 25 parts, among them J14 Volume, J15 Left Speaker, Q1 AOD417, U4 MAX9744

Commit message: isolating 12v and amp from microcontroller
Parts:
- added C11: 10µF, Capacitor_SMD:C_0805_2012Metric_Pad1.15x1.40mm_HandSolder, symbol Device:C
- added U3: AP2112K-3.3, Package_TO_SOT_SMD:SOT-23-5, symbol Regulator_Linear:AP2112K-3.3
Connections:
- net GND: now also C11.2, U3.2 (GND)
- net at C3.1, C4.2, C5.2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: now also U3.1 (VIN), U3.3 (EN)
- net +3V3 renamed +3.3VP
- net +3.3VP: now also C11.1, U3.5 (VOUT)
Other:
- moved on the sheet: C1, C10, C12, C13, C2, C3, C4, C5, C6, C7, C8, C9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
