File: hardware/InputBoardSTM32/InputBoardSTM32.sch (KiCad schematic (older format))
At the start: 16 parts, among them J1 8P8C, J10 Conn_01x04_Male, J11 Conn_01x04_Male, J2 Conn_01x04_Male, J3 Conn_01x04_Male, J4 Conn_ARM_JTAG_SWD_10, J5 Conn_01x04_Male, J6 Conn_01x04_Male, J7 Conn_01x04_Male, J9 Conn_01x04_Male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

Commit message: InputBoardSTM32 V1 complete
Parts:
- J1: footprint Useful Modifications:RJ45_x08_Horizontal_tabs -> Useful Modifications:RJ45_x08_Tab_Up
- J2: footprint Connector_JST:JST_SH_SM04B-SRSS-TB_1x04-1MP_P1.00mm_Horizontal -> Connector_JST:JST_SH_BM04B-SRSS-TB_1x04-1MP_P1.00mm_Vertical
- J3: footprint Connector_PinHeader_2.54mm:PinHeader_1x04_P2.54mm_Vertical -> Connector_JST:JST_SH_BM04B-SRSS-TB_1x04-1MP_P1.00mm_Vertical
- J4: footprint (none) -> Useful Modifications:JTAG_SWD_SMD
Connections:
- net +3V3: now also J3.2 (Pin_2); no longer J3.1 (Pin_1)
- net GND: now also J3.1 (Pin_1); no longer J3.2 (Pin_2)
- no-connect marks 2 -> 6
Other:
- moved on the sheet: J3
Changed lines of the file:
@@
 F 0 "J1" V 4201 2100 50  0000 L CNN
 F 1 "8P8C" V 4292 2100 50  0000 L CNN
-F 2 "Useful Modifications:RJ45_x08_Horizontal_tabs" V 4190 1595 50  0001 C CNN
+F 2 "Useful Modifications:RJ45_x08_Tab_Up" V 4190 1595 50  0001 C CNN
 F 3 "~" V 4190 1595 50  0001 C CNN
 	1    4190 1570
@@
 F 0 "J2" H 8998 4071 50  0000 C CNN
 F 1 "Conn_01x04_Male" H 8998 3980 50  0000 C CNN
-F 2 "Connector_JST:JST_SH_SM04B-SRSS-TB_1x04-1MP_P1.00mm_Horizontal" H 8890 3790 50  0001 C CNN
+F 2 "Connector_JST:JST_SH_BM04B-SRSS-TB_1x04-1MP_P1.00mm_Vertical" H 8890 3790 50  0001 C CNN
 F 3 "~" H 8890 3790 50  0001 C CNN
 	1    8890 3790
@@
 L Connector:Conn_01x04_Male J3
 U 1 1 604F8C23
-P 6210 3920
-F 0 "J3" H 6318 4201 50  0000 C CNN
-F 1 "Conn_01x04_Male" H 6318 4110 50  0000 C CNN
-F 2 "Connector_PinHeader_2.54mm:PinHeader_1x04_P2.54mm_Vertical" H 6210 3920 50  0001 C CNN
-F 3 "~" H 6210 3920 50  0001 C CNN
-	1    6210 3920
+P 6150 3900
+F 0 "J3" H 6258 4181 50  0000 C CNN
+F 1 "Conn_01x04_Male" H 6258 4090 50  0000 C CNN
+F 2 "Connector_JST:JST_SH_BM04B-SRSS-TB_1x04-1MP_P1.00mm_Vertical" H 6150 3900 50  0001 C CNN
+F 3 "~" H 6150 3900 50  0001 C CNN
+	1    6150 3900
 	1    0    0    -1
 $EndComp
@@
 L power:GND #PWR01
 U 1 1 604FB52D
-P 6410 3920
-F 0 "#PWR01" H 6410 3670 50  0001 C CNN
-F 1 "GND" V 6410 3720 50  0000 C CNN
-F 2 "" H 6410 3920 50  0001 C CNN
-F 3 "" H 6410 3920 50  0001 C CNN
-	1    6410 3920
+P 6350 3800
+F 0 "#PWR01" H 6350 3550 50  0001 C CNN
+F 1 "GND" V 6350 3600 50  0000 C CNN
+F 2 "" H 6350 3800 50  0001 C CNN
+F 3 "" H 6350 3800 50  0001 C CNN
+	1    6350 3800
 	0    -1   -1   0
 $EndComp
@@
 L power:+3.3V #PWR02
 U 1 1 604FBE91
-P 6410 3820
-F 0 "#PWR02" H 6410 3670 50  0001 C CNN
-F 1 "+3.3V" V 6410 4080 50  0000 C CNN
-F 2 "" H 6410 3820 50  0001 C CNN
-F 3 "" H 6410 3820 50  0001 C CNN
-	1    6410 3820
-	0    1    1    0
-$EndComp
-Text GLabel 6410 4020 2    50   Input ~ 0
+P 6350 3900
+F 0 "#PWR02" H 6350 3750 50  0001 C CNN
+F 1 "+3.3V" V 6350 4160 50  0000 C CNN
+F 2 "" H 6350 3900 50  0001 C CNN
+F 3 "" H 6350 3900 50  0001 C CNN
+	1    6350 3900
+	0    1    1    0
+$EndComp
+Text GLabel 6350 4000 2    50   Input ~ 0
 TX
-Text GLabel 6410 4120 2    50   Input ~ 0
+Text GLabel 6350 4100 2    50   Input ~ 0
 RX
 $Comp
@@
 F 0 "J4" H 3957 3996 50  0000 R CNN
 F 1 "Conn_ARM_JTAG_SWD_10" H 3957 3905 50  0000 R CNN
-F 2 "" H 4400 3950 50  0001 C CNN
+F 2 "Useful Modifications:JTAG_SWD_SMD" H 4400 3950 50  0001 C CNN
 F 3 "http://infocenter.arm.com/help/topic/com.arm.doc.ddi0314h/DDI0314H_coresight_components_trm.pdf" V 4050 2700 50  0001 C CNN
 	1    4400 3950
@@
 Connection ~ 4350 4650
 NoConn ~ 4900 4050
+NoConn ~ 7150 2000
+NoConn ~ 7150 2100
+NoConn ~ 7150 1500
+NoConn ~ 5750 1500
 $EndSCHEMATC
