File: hardware/InputBoardSTM32QFN28/InputBoardSTM32QFN28.sch (KiCad schematic (older format))
At the start: 16 parts, among them J1 8P8C, J10 Conn_01x04_Male, J11 Conn_01x04_Male, J2 Conn_01x04_Male, J3 Conn_01x04_Male, J4 Conn_ARM_JTAG_SWD_10, J5 Conn_01x04_Male, J6 Conn_01x04_Male, J7 Conn_01x04_Male, J9 Conn_01x04_Male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

Commit message: updates to STM32 Input PCB and new STM32 QFN28 Input PCB
Parts:
- added C4: 100nF, Capacitor_SMD:C_0805_2012Metric, symbol Device:C_Small
- added Y1: ECS-3225MVQ-160-BP-TR, Useful Modifications:OSC_ECS-3225MVQ-160-BP-TR, symbol CrystalOscillator:ECS-3225MVQ-160-BP-TR
- U1: footprint Package_SO:TSSOP-20_4.4x6.5mm_P0.65mm -> Useful Modifications:STM32G031G8U6; symbol STM32:STM32G031F4Px -> STM32QFN:STM32G031G8U6
Connections:
- net labels added: OscillatorIn
- wire segments 15 -> 19
- no-connect marks 6 -> 3
Other:
- note added: "Power\nCapacitors"
- note added: "STM32 Crystal Oscillator"
- moved on the sheet: C1, C2, C3, J1
