File: hardware/Pitt State/Two Motor Nano Controller/Two Motor Nano Controller.sch (KiCad schematic (older format))
At the start: 12 parts, among them J1 Additiona Inputs Front, J10 Limit Switch Front, J2 Stepper Minus Front, J3 Stepper Plus Front, J4 Limit Switch Front, J5 12v Power, J6 Analog Steering, J7 Additiona Inputs Back, J8 Stepper Minus Front, J9 Stepper Plus Back

Commit message: updated Pitt State PCBs
Parts:
- J6: footprint Project:TerminalBlock_bornier-2_P5.08mm -> Project:JST_XH_B2B-XH-A_1x02_P2.54mm_Vertical
Changed lines of the file:
@@
 F 0 "J6" H 5553 5171 50  0000 L CNN
 F 1 "Analog Steering" H 5553 5080 50  0000 L CNN
-F 2 "Project:TerminalBlock_bornier-2_P5.08mm" H 5525 5195 50  0001 C CNN
+F 2 "Project:JST_XH_B2B-XH-A_1x02_P2.54mm_Vertical" H 5525 5195 50  0001 C CNN
 F 3 "~" H 5525 5195 50  0001 C CNN
 	1    5525 5195
