File: hardware/DriveByWireInputAltSTM32QFN28/DriveByWireInputAltSTM32QFN28.kicad_pcb (KiCad board)
At the start: 2 copper layers, 39.7 x 29.4 mm, 16 parts, among them J1 8P8C, J2 Conn_01x04_Male, J3 Conn_01x04_Male, J4 Conn_ARM_JTAG_SWD_10, J5 Conn_01x02_Male, J6 Conn_01x02_Male, U1 STM32G031F4Px, Y1 ECS-3225MVQ-160-BP-TR

Commit message: finalizing drive-by-wire PCBs
Parts:
- J4: value Conn_ARM_JTAG_SWD_10 -> Conn_01x05_Male; footprint Useful Modifications:JTAG_SWD_SMD -> Connector_JST:JST_SH_BM05B-SRSS-TB_1x05-1MP_P1.00mm_Vertical
- moved J4 0.86 mm to (167.6, 101.8), turned to -90 degrees
Connections:
- J4 pad 2: SWDIO -> GND
- J4 pad 3: GND -> SWCLK
- J4 pad 4: SWCLK -> SWDIO
- J4 pad 5: GND -> /RESET
Routing:
- net GND: track 20.1 -> 23.1 mm, vias 19 -> 20
- net SWCLK: track 28.8 -> 31.8 mm
- net SWDIO: track 22.7 -> 25.6 mm
- net /RESET: track 60.7 -> 58.5 mm
Other:
- board text added: "Drive-by-Wire Alt V1"
- board text removed: "Drive-by-Wire V1"

Commit message: Drive by wire PCB Gerbers
Other:
- board text added: "SWD"
Changed lines of the file:
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@@
     (effects (font (size 0.6 0.6) (thickness 0.1)))
+  )
+  (gr_text "SWD" (at 167.66 96.4) (layer "F.SilkS")
+    (effects (font (size 0.75 0.75) (thickness 0.13)))
   )
   (gr_text "Sound 2" (at 157.49 86.35) (layer "F.SilkS")
