File: hardware/DriveByWireInputSTM32QFN28/DriveByWireInputSTM32QFN28.kicad_pcb (KiCad board)
At the start: 2 copper layers, 39.7 x 29.4 mm, 16 parts, among them J1 8P8C, J2 Conn_01x04_Male, J3 Conn_01x04_Male, J4 Conn_ARM_JTAG_SWD_10, J5 Conn_01x02_Male, J6 Conn_01x02_Male, U1 STM32G031F4Px, Y1 ECS-3225MVQ-160-BP-TR

Commit message: Drive by wire PCB Gerbers
Other:
- board text added: "SWD"
Changed lines of the file:
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@@
+    (effects (font (size 0.75 0.75) (thickness 0.13)))
+  )
+  (gr_text "SWD" (at 161.56 100.28) (layer "F.SilkS")
     (effects (font (size 0.75 0.75) (thickness 0.13)))
   )
