File: hardware/InputJoyStickSTM32QFN28/InputJoyStickSTM32QFN28.kicad_sch (KiCad schematic)
At the start: 17 parts, among them J1 8P8C, J2 Conn_01x04_Male, J3 Conn_01x04_Male, J4 Conn_ARM_JTAG_SWD_10, J5 Conn_01x05_Male, J6 Conn_01x02_Male, J7 Conn_01x02_Male, J8 Conn_01x02_Male, J9 Conn_01x02_Male, U1 STM32G031F4Px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

Commit message: Updating Input Joystick PCB to add additional LED connector and switch to Tag-Connect for programming
Parts:
- removed J4: Conn_ARM_JTAG_SWD_10, Useful Modifications:JTAG_SWD_SMD, symbol Connector:Conn_ARM_JTAG_SWD_10
- added D1: LED_Small, LED_SMD:LED_0603_1608Metric, symbol Device:LED_Small
- added J10: Conn_01x02_Male, Connector_JST:JST_XH_B2B-XH-A_1x02_P2.50mm_Vertical, symbol Connector:Conn_01x02_Male
- added J4: TagConnect_TC2030-NL, Connector:Tag-Connect_TC2030-IDC-NL_2x03_P1.27mm_Vertical, symbol Connector:Conn_ARM_SWD_TagConnect_TC2030-NL
- added R3: 470, Resistor_SMD:R_0603_1608Metric, symbol Device:R_Small
- C1, C2, C4: MPN (none) -> C49678
- C3: MPN (none) -> C15850
- J2, J3: MPN (none) -> C145961
- R1, R2: footprint Resistor_SMD:R_0805_2012Metric_Pad1.15x1.40mm_HandSolder -> Resistor_SMD:R_0805_2012Metric; MPN (none) -> C17414
- U1: MPN (none) -> C432211
- Y1: MPN (none) -> C252336
Connections:
- net +3V3: now also J4.1 (VCC)
- net +5V: now also J10.1 (Pin_1)
- net GND: now also D1.1 (K), J10.2 (Pin_2), J4.5 (GND)
- net RESET: now also J4.3 (~{RESET})
- net SWCLK: now also J4.4 (SWCLK)
- net SWDIO: now also J4.2 (SWDIO)
- net USER_LED: now reaches U1.22 (PA15)
- net USER_LED: now also R3.2
- new net: D1.2 (A), R3.1
- no-connect marks 3 -> 10
Other:
- note added: "LEDs"
- note removed: "Sound Buttons do not connect to the microcontroller."
- moved on the sheet: C1, J7, J9, U1
