File: hardware/ControlPanelSTM32QFN28/ControlPanelSTM32QFN28.kicad_pcb (KiCad board)
At the start: 2 copper layers, 45 x 29.4 mm, 22 parts, among them J1 8P8C, J10 Conn_01x04_Male, J11 Conn_01x04_Male, J12 Conn_01x02_Male, J13 Conn_01x02_Male, J14 Conn_01x02_Male, J15 Conn_01x02_Male, J4 Conn_02x03, J5 Conn_01x04_Male, J6 Conn_01x04_Male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

Commit message: moving pcb file and generating gerbers
Parts:
- moved C3 11.3 mm to (142.5, 103.2), turned to 180 degrees
- moved C4 5.68 mm to (157.4, 98.1), turned to 180 degrees
- moved C2 3.46 mm to (143.2, 96.6)
- moved Y1 2.44 mm to (153.5, 98.5), turned to 90 degrees
- moved U1 1.91 mm to (147.9, 98.7)
- moved C1 1.41 mm to (142.5, 100.0), turned to 0 degrees
Routing:
- net LeftButton: track 0.00 -> 19.7 mm, vias 0 -> 1
- net ReverseButton: track 0.00 -> 17.3 mm, vias 0 -> 1
- net DriveButton: track 0.00 -> 13.9 mm, vias 0 -> 1
- net RightButton: track 0.00 -> 13.5 mm, vias 0 -> 1
- net JoyX: track 0.00 -> 10.9 mm, vias 0 -> 1
- net +3V3: track 27.2 -> 34.5 mm
- net GND: track 2.72 -> 9.09 mm, vias 3 -> 1
- net JoyY: track 0.00 -> 4.88 mm, vias 0 -> 1
- net SWDIO: track 11.3 -> 15.7 mm
- net SWCLK: track 16.3 -> 19.5 mm
- net OscillatorIn: track 2.56 -> 5.26 mm
- net +5V: track 45.4 -> 43.6 mm
- net Other: track 2.69 -> 4.45 mm
- net /RESET: track 15.4 -> 16.1 mm
Other:
- board text removed: "3v"
- board text removed: "Gnd"
- board text removed: "S"

Commit message: updating control panel PCB to KiCad 6
Other:
- net class Default removed

Commit message: updating control panel PCB to use new programming header, smaller SMDs and with JLCPCB part numbers
Parts:
- removed J4: Conn_02x03, Connector_PinHeader_2.54mm:PinHeader_2x03_P2.54mm_Vertical
- added D1: LED_Small, Capacitor_SMD:C_0603_1608Metric, F.Cu at (135.4, 105.3)
- added J2: TagConnect_TC2030-NL, Connector:Tag-Connect_TC2030-IDC-NL_2x03_P1.27mm_Vertical, F.Cu at (135.3, 100.1)
- added R1: 470, Capacitor_SMD:C_0402_1005Metric, B.Cu at (143.6, 101.7)
- C1, C2, C4: footprint Capacitor_SMD:C_0805_2012Metric -> Capacitor_SMD:C_0402_1005Metric
- C3: footprint Capacitor_SMD:C_0805_2012Metric -> Capacitor_SMD:C_0603_1608Metric
- moved C3 13.8 mm to (153.9, 95.5)
- moved C1 9.15 mm to (151.6, 101.0)
- moved C2 8.08 mm to (151.2, 95.3), turned to 0 degrees
- moved C4 0.82 mm to (156.9, 97.4)
- turned Y1 to 180 degrees
Connections:
- J10 pad 2: Sound1 -> Sound2
- J11 pad 2: Sound2 -> Sound1
- U1 pad 10: Net-(U1-Pad10) -> unconnected-(U1-PA4-Pad10)
- U1 pad 13: Net-(U1-Pad13) -> unconnected-(U1-PA7-Pad13)
- U1 pad 16: Net-(U1-Pad16) -> unconnected-(U1-PA8-Pad16)
- U1 pad 2: Net-(U1-Pad2) -> unconnected-(U1-PC15-OSC32_OUT-Pad2)
- U1 pad 22: Net-(U1-Pad22) -> unconnected-(U1-PA15-Pad22)
- U1 pad 23: Net-(U1-Pad23) -> unconnected-(U1-PB3-Pad23)
- U1 pad 24: Net-(U1-Pad24) -> unconnected-(U1-PB4-Pad24)
- U1 pad 25: Net-(U1-Pad25) -> unconnected-(U1-PB5-Pad25)
- U1 pad 26: Net-(U1-Pad26) -> unconnected-(U1-PB6-Pad26)
- U1 pad 27: Net-(U1-Pad27) -> unconnected-(U1-PB7-Pad27)
- U1 pad 28: Net-(U1-Pad28) -> unconnected-(U1-PB8-Pad28)
- U1 pad 6: Net-(U1-Pad6) -> unconnected-(U1-PA0-Pad6)
- U1 pad 7: Net-(U1-Pad7) -> unconnected-(U1-PA1-Pad7)
- U1 pad 8: Net-(U1-Pad8) -> USER_LED
- U1 pad 9: Net-(U1-Pad9) -> unconnected-(U1-PA3-Pad9)
- Y1 pad 1: Net-(Y1-Pad1) -> unconnected-(Y1-TRI-STATE-Pad1)
Routing:
- net +3V3: track 34.5 -> 58.4 mm, vias 2 -> 1
- net Sound1: track 26.6 -> 39.8 mm
- net Sound2: track 34.3 -> 24.3 mm
- net Net-(D1-A): track 0.00 -> 8.48 mm, vias 0 -> 1
- net USER_LED: track 0.00 -> 7.86 mm, vias 0 -> 2
- net SWDIO: track 15.7 -> 21.5 mm, vias 0 -> 1
- net /RESET: track 16.1 -> 21.0 mm, vias 2 -> 1
- net OscillatorIn: track 5.26 -> 2.51 mm
- net GND: track 9.09 -> 10.8 mm, vias 1 -> 15
- net SWCLK: track 19.5 -> 18.1 mm, vias 0 -> 1
- net RightButton: track 13.5 -> 14.5 mm
- net JoyY: track 4.88 -> 5.64 mm, vias 1 -> 0
- net LeftButton: track 19.7 -> 20.3 mm
- net ReverseButton: track 17.3 -> 17.8 mm, vias 1 -> 0
- net JoyX: track 10.9 -> 10.7 mm, vias 1 -> 0
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Other:
- board text added: "+"
- board text added: "Gnd"
- board text added: "Input Board STM32QFN28 v2"
- board text added: "Programming"
- board text added: "S2 S1"
- board text added: "User LED"
- board text added: "V2"
- board text removed: "Input Board STM32QFN28 v1"
- board text removed: "S1 S2"
- board text removed: "V1"
