File: hardware/motor-controller-v3/motor-controller-v3.kicad_sch (KiCad schematic)
At the start: 63 parts, among them J101 WAGO, J102 WAGO, J103 2.54mm R/A, J104 WAGO, J105 WAGO, J106 WAGO, Q101 AO3401A, Q102 AO3401A, Q103 AO3401A, Q104 AO3400A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

Commit message: Finished motor-controller-v3 draft
Parts:
- H101, H102, H103, H104: value M3 -> M2.5; footprint MountingHole:MountingHole_3.2mm_M3_Pad_Via -> MountingHole:MountingHole_2.7mm_M2.5_Pad_Via
- H105, H106: value M2.5 -> M2; footprint MountingHole:MountingHole_2.7mm_M2.5_Pad_Via -> MountingHole:MountingHole_2.2mm_M2_Pad_Via
- R106, R109, R111: value 4.7kΩ -> 130Ω; MPN C23162 -> C22796
- R113: value 4.7kΩ -> 56Ω; MPN C23162 -> C25196
Changed lines of the file:
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@@
 		)
 	)
-	(text_box "UPDATE SERIES RESISTOR VALUES!"
-		(exclude_from_sim no)
-		(at 321.31 208.28 0)
-		(size 63.5 3.81)
-		(margins 0.9525 0.9525 0.9525 0.9525)
-		(stroke
-			(width 0)
-			(type solid)
-			(color 255 4 0 1)
-		)
-		(fill
-			(type color)
-			(color 255 239 0 1)
-		)
-		(effects
-			(font
-				(size 1.27 1.27)
-				(color 255 37 1 1)
-			)
-		)
-	)
 	(junction
 		(at 73.66 123.19)
@@
 			)
 		)
-		(property "Value" "4.7kΩ"
+		(property "Value" "130Ω"
 			(at 341.63 184.1499 0)
 			(effects
@@
 			)
 		)
-		(property "Datasheet" "https://www.lcsc.com/datasheet/C23162.pdf"
+		(property "Datasheet" "https://www.lcsc.com/datasheet/C22796.pdf"
 			(at 339.09 182.88 0)
 			(effects
@@
 			)
 		)
-		(property "Description" "RES 4.7kΩ ±1% 100mW 0603"
+		(property "Description" "RES 130Ω ±1% 100mW 0603"
 			(at 339.09 182.88 0)
 			(effects
@@
 			)
 		)
-		(property "MPN" "C23162"
+		(property "MPN" "C22796"
 			(at 339.09 182.88 0)
 			(effects
@@
 			)
 		)
-		(property "Value" "M2.5"
+		(property "Value" "M2"
 			(at 212.09 243.8399 0)
 			(effects
@@
 			)
 		)
-		(property "Footprint" "MountingHole:MountingHole_2.7mm_M2.5_Pad_Via"
+		(property "Footprint" "MountingHole:MountingHole_2.2mm_M2_Pad_Via"
 			(at 209.55 243.84 0)
 			(effects
@@
 			)
 		)
-		(property "Value" "M3"
+		(property "Value" "M2.5"
 			(at 166.37 243.8399 0)
 			(effects
@@
 			)
 		)
-		(property "Footprint" "MountingHole:MountingHole_3.2mm_M3_Pad_Via"
+		(property "Footprint" "MountingHole:MountingHole_2.7mm_M2.5_Pad_Via"
 			(at 163.83 243.84 0)
 			(effects
@@
 			)
 		)
-		(property "Value" "M3"
+		(property "Value" "M2.5"
 			(at 189.23 243.8399 0)
 			(effects
@@
 			)
 		)
-		(property "Footprint" "MountingHole:MountingHole_3.2mm_M3_Pad_Via"
+		(property "Footprint" "MountingHole:MountingHole_2.7mm_M2.5_Pad_Via"
 			(at 186.69 243.84 0)
 			(effects
@@
 	)
 	(symbol
+		(lib_id "Device:R_US")
+		(at 386.08 130.81 0)
+		(unit 1)
+		(exclude_from_sim no)
+		(in_bom yes)
+		(on_board yes)
+		(dnp no)
+		(property "Reference" "R106"
+			(at 388.62 129.5399 0)
+			(effects
+				(font
+					(size 1.27 1.27)
+				)
+				(justify left)
+			)
+		)
+		(property "Value" "130Ω"
+			(at 388.62 132.0799 0)
+			(effects
+				(font
+					(size 1.27 1.27)
+				)
+				(justify left)
+			)
+		)
+		(property "Footprint" "Resistor_SMD:R_0603_1608Metric"
+			(at 387.096 131.064 90)
+			(effects
+				(font
+					(size 1.27 1.27)
+				)
+				(hide yes)
+			)
+		)
+		(property "Datasheet" "https://www.lcsc.com/datasheet/C22796.pdf"
+			(at 386.08 130.81 0)
+			(effects
+				(font
+					(size 1.27 1.27)
+				)
+				(hide yes)
+			)
+		)
+		(property "Description" "RES 130Ω ±1% 100mW 0603"
+			(at 386.08 130.81 0)
+			(effects
+				(font
+					(size 1.27 1.27)
+				)
+				(hide yes)
+			)
+		)
+		(property "MPN" "C22796"
+			(at 386.08 130.81 0)
+			(effects
+				(font
+					(size 1.27 1.27)
+				)
+				(hide yes)
+			)
+		)
+		(pin "1"
+		)
+		(pin "2"
+		)
+		(instances
+			(project "motor-controller-v3"
+				(path "/8badd534-6f39-4fa0-90cd-9d3408a5706c"
+					(reference "R106")
+					(unit 1)
+				)
+			)
+		)
+	)
+	(symbol
 		(lib_id "Connector:TestPoint")
 		(at 67.31 77.47 270)
@@
 			)
 		)
-		(property "Value" "4.7kΩ"
+		(property "Value" "56Ω"
 			(at 341.63 129.5399 0)
 			(effects
@@
 			)
 		)
-		(property "Datasheet" "https://www.lcsc.com/datasheet/C23162.pdf"
+		(property "Datasheet" "https://www.lcsc.com/datasheet/C25196.pdf"
 			(at 339.09 128.27 0)
 			(effects
@@
 			)
 		)
-		(property "Description" "RES 4.7kΩ ±1% 100mW 0603"
+		(property "Description" "RES 56Ω ±1% 100mW 0603"
 			(at 339.09 128.27 0)
 			(effects
@@
 			)
 		)
-		(property "MPN" "C23162"
+		(property "MPN" "C25196"
 			(at 339.09 128.27 0)
 			(effects
@@
 			)
 		)
-		(property "Value" "M3"
+		(property "Value" "M2.5"
 			(at 154.94 243.8399 0)
 			(effects
@@
 			)
 		)
-		(property "Footprint" "MountingHole:MountingHole_3.2mm_M3_Pad_Via"
+		(property "Footprint" "MountingHole:MountingHole_2.7mm_M2.5_Pad_Via"
 			(at 152.4 243.84 0)
 			(effects
@@
 			)
 		)
-		(property "Value" "M3"
+		(property "Value" "M2.5"
 			(at 177.8 243.8399 0)
 			(effects
@@
 			)
 		)
-		(property "Footprint" "MountingHole:MountingHole_3.2mm_M3_Pad_Via"
+		(property "Footprint" "MountingHole:MountingHole_2.7mm_M2.5_Pad_Via"
 			(at 175.26 243.84 0)
 			(effects
@@
 	)
 	(symbol
-		(lib_id "Device:R_US")
-		(at 386.08 130.81 0)
-		(unit 1)
-		(exclude_from_sim no)
-		(in_bom yes)
-		(on_board yes)
-		(dnp no)
-		(property "Reference" "R106"
-			(at 388.62 129.5399 0)
-			(effects
-				(font
-					(size 1.27 1.27)
-				)
-				(justify left)
-			)
-		)
-		(property "Value" "4.7kΩ"
-			(at 388.62 132.0799 0)
-			(effects
-				(font
-					(size 1.27 1.27)
-				)
-				(justify left)
-			)
-		)
-		(property "Footprint" "Resistor_SMD:R_0603_1608Metric"
-			(at 387.096 131.064 90)
-			(effects
-				(font
-					(size 1.27 1.27)
-				)
-				(hide yes)
-			)
-		)
-		(property "Datasheet" "https://www.lcsc.com/datasheet/C23162.pdf"
-			(at 386.08 130.81 0)
-			(effects
-				(font
-					(size 1.27 1.27)
-				)
-				(hide yes)
-			)
-		)
-		(property "Description" "RES 4.7kΩ ±1% 100mW 0603"
-			(at 386.08 130.81 0)
-			(effects
-				(font
-					(size 1.27 1.27)
-				)
-				(hide yes)
-			)
-		)
-		(property "MPN" "C23162"
-			(at 386.08 130.81 0)
-			(effects
-				(font
-					(size 1.27 1.27)
-				)
-				(hide yes)
-			)
-		)
-		(pin "1"
-		)
-		(pin "2"
-		)
-		(instances
-			(project "motor-controller-v3"
-				(path "/8badd534-6f39-4fa0-90cd-9d3408a5706c"
-					(reference "R106")
-					(unit 1)
-				)
-			)
-		)
-	)
-	(symbol
 		(lib_id "power:GND")
 		(at 386.08 196.85 0)
@@
 			)
 		)
-		(property "Value" "M2.5"
+		(property "Value" "M2"
 			(at 200.66 243.8399 0)
 			(effects
@@
 			)
 		)
-		(property "Footprint" "MountingHole:MountingHole_2.7mm_M2.5_Pad_Via"
+		(property "Footprint" "MountingHole:MountingHole_2.2mm_M2_Pad_Via"
 			(at 198.12 243.84 0)
 			(effects
@@
 			)
 		)
-		(property "Value" "4.7kΩ"
+		(property "Value" "130Ω"
 			(at 388.62 184.1499 0)
 			(effects
@@
 			)
 		)
-		(property "Datasheet" "https://www.lcsc.com/datasheet/C23162.pdf"
+		(property "Datasheet" "https://www.lcsc.com/datasheet/C22796.pdf"
 			(at 386.08 182.88 0)
 			(effects
@@
 			)
 		)
-		(property "Description" "RES 4.7kΩ ±1% 100mW 0603"
+		(property "Description" "RES 130Ω ±1% 100mW 0603"
 			(at 386.08 182.88 0)
 			(effects
@@
 			)
 		)
-		(property "MPN" "C23162"
+		(property "MPN" "C22796"
 			(at 386.08 182.88 0)
 			(effects

Commit message: Adjust R_sense
Parts:
- TP101, TP102, TP103, TP104, TP105, TP106, TP107, TP108, TP109, TP110, TP111, TP112, TP113, TP114, TP115, TP116, TP117, TP118, TP119, TP120, TP121, TP124, TP125, TP126: now left out of the parts list
Changed lines of the file:
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@@
 		)
 	)
+	(text_box "NOTE: ADJUST R_{SENSE} AND V_{REF} DIVIDER VALUES BASED ON EXPECTED STALL CURRENT!"
+		(exclude_from_sim no)
+		(at 185.42 91.44 0)
+		(size 48.26 5.08)
+		(margins 0.9525 0.9525 0.9525 0.9525)
+		(stroke
+			(width 0)
+			(type solid)
+			(color 255 11 0 1)
+		)
+		(fill
+			(type color)
+			(color 255 245 0 1)
+		)
+		(effects
+			(font
+				(size 1.27 1.27)
+				(color 255 2 0 1)
+			)
+		)
+	)
 	(junction
 		(at 73.66 123.19)
@@
 		(unit 1)
 		(exclude_from_sim no)
-		(in_bom yes)
+		(in_bom no)
 		(on_board yes)
 		(dnp no)
@@
 		(unit 1)
 		(exclude_from_sim no)
-		(in_bom yes)
+		(in_bom no)
 		(on_board yes)
 		(dnp no)
@@
 		(unit 1)
 		(exclude_from_sim no)
-		(in_bom yes)
+		(in_bom no)
 		(on_board yes)
 		(dnp no)
@@
 		(unit 1)
 		(exclude_from_sim no)
-		(in_bom yes)
+		(in_bom no)
 		(on_board yes)
 		(dnp no)
@@
 		(unit 1)
 		(exclude_from_sim no)
-		(in_bom yes)
+		(in_bom no)
 		(on_board yes)
 		(dnp no)
@@
 		(unit 1)
 		(exclude_from_sim no)
-		(in_bom yes)
+		(in_bom no)
 		(on_board yes)
 		(dnp no)
@@
 		(unit 1)
 		(exclude_from_sim no)
-		(in_bom yes)
+		(in_bom no)
 		(on_board yes)
 		(dnp no)
@@
 		(unit 1)
 		(exclude_from_sim no)
-		(in_bom yes)
+		(in_bom no)
 		(on_board yes)
 		(dnp no)
@@
 		(unit 1)
 		(exclude_from_sim no)
-		(in_bom yes)
+		(in_bom no)
 		(on_board yes)
 		(dnp no)
@@
 		(unit 1)
 		(exclude_from_sim no)
-		(in_bom yes)
+		(in_bom no)
 		(on_board yes)
 		(dnp no)
@@
 		(unit 1)
 		(exclude_from_sim no)
-		(in_bom yes)
+		(in_bom no)
 		(on_board yes)
 		(dnp no)
@@
 		(unit 1)
 		(exclude_from_sim no)
-		(in_bom yes)
+		(in_bom no)
 		(on_board yes)
 		(dnp no)
@@
 		(unit 1)
 		(exclude_from_sim no)
-		(in_bom yes)
+		(in_bom no)
 		(on_board yes)
 		(dnp no)
@@
 		(unit 1)
 		(exclude_from_sim no)
-		(in_bom yes)
+		(in_bom no)
 		(on_board yes)
 		(dnp no)
@@
 		(unit 1)
 		(exclude_from_sim no)
-		(in_bom yes)
+		(in_bom no)
 		(on_board yes)
 		(dnp no)
@@
 		(unit 1)
 		(exclude_from_sim no)
-		(in_bom yes)
+		(in_bom no)
 		(on_board yes)
 		(dnp no)
@@
 		(unit 1)
 		(exclude_from_sim no)
-		(in_bom yes)
+		(in_bom no)
 		(on_board yes)
 		(dnp no)
@@
 		(unit 1)
 		(exclude_from_sim no)
-		(in_bom yes)
+		(in_bom no)
 		(on_board yes)
 		(dnp no)
@@
 		(unit 1)
 		(exclude_from_sim no)
-		(in_bom yes)
+		(in_bom no)
 		(on_board yes)
 		(dnp no)
@@
 		(unit 1)
 		(exclude_from_sim no)
-		(in_bom yes)
+		(in_bom no)
 		(on_board yes)
 		(dnp no)
@@
 		(unit 1)
 		(exclude_from_sim no)
-		(in_bom yes)
+		(in_bom no)
 		(on_board yes)
 		(dnp no)
@@
 		(unit 1)
 		(exclude_from_sim no)
-		(in_bom yes)
+		(in_bom no)
 		(on_board yes)
 		(dnp no)
@@
 		(unit 1)
 		(exclude_from_sim no)
-		(in_bom yes)
+		(in_bom no)
 		(on_board yes)
 		(dnp no)
@@
 		(unit 1)
 		(exclude_from_sim no)
-		(in_bom yes)
+		(in_bom no)
 		(on_board yes)
 		(dnp no)
