File: hardware/RyderSteeringButtonConnector/RyderSteeringButtonConnector.kicad_sch (KiCad schematic)
At the start: 7 parts, among them J1 Conn_01x04_Pin, J2 Conn_01x05_Pin, J3 Conn_01x03_Pin, J4 Conn_01x03_Pin, J5 Conn_01x03_Pin

Commit message: v2 of ryder steering wheel button connnector pcb
Parts:
- J3, J4, J5: footprint Connector_JST:JST_SH_SM03B-SRSS-TB_1x03-1MP_P1.00mm_Horizontal -> Connector_JST:JST_SH_BM03B-SRSS-TB_1x03-1MP_P1.00mm_Vertical; LCSC Part # C160403 -> C160389
Changed lines of the file:
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@@
 			)
 		)
-		(property "Footprint" "Connector_JST:JST_SH_SM03B-SRSS-TB_1x03-1MP_P1.00mm_Horizontal"
+		(property "Footprint" "Connector_JST:JST_SH_BM03B-SRSS-TB_1x03-1MP_P1.00mm_Vertical"
 			(at 205.74 97.79 0)
 			(effects
@@
 			)
 		)
-		(property "LCSC Part #" "C160403"
+		(property "LCSC Part #" "C160389"
 			(at 205.74 97.79 0)
 			(effects
@@
 			)
 		)
-		(property "Footprint" "Connector_JST:JST_SH_SM03B-SRSS-TB_1x03-1MP_P1.00mm_Horizontal"
+		(property "Footprint" "Connector_JST:JST_SH_BM03B-SRSS-TB_1x03-1MP_P1.00mm_Vertical"
 			(at 179.07 97.79 0)
 			(effects
@@
 			)
 		)
-		(property "LCSC Part #" "C160403"
+		(property "LCSC Part #" "C160389"
 			(at 179.07 97.79 0)
 			(effects
@@
 			)
 		)
-		(property "Footprint" "Connector_JST:JST_SH_SM03B-SRSS-TB_1x03-1MP_P1.00mm_Horizontal"
+		(property "Footprint" "Connector_JST:JST_SH_BM03B-SRSS-TB_1x03-1MP_P1.00mm_Vertical"
 			(at 148.59 97.79 0)
 			(effects
@@
 			)
 		)
-		(property "LCSC Part #" "C160403"
+		(property "LCSC Part #" "C160389"
 			(at 148.59 97.79 0)
 			(effects
