File: hardware/Ryder/geeks-ecu/DRV8701.kicad_sch (KiCad schematic)
At the start: 20 parts, among them Q601 60V 45A, Q602 60V 45A, Q603 60V 45A, Q605 60V 45A, U501 DRV8701P

Commit message: Ryder ECU Cleanup
Still need to work on high current traces
Parts:
- C601: renamed from C501; footprint Capacitor_SMD:C_0603_1608Metric -> geeks-ecu-footprints:C_0603_1608Metric
- C602: renamed from C502; footprint Capacitor_SMD:C_0603_1608Metric -> geeks-ecu-footprints:C_0603_1608Metric
- C603: renamed from C503; footprint Capacitor_SMD:C_0603_1608Metric -> geeks-ecu-footprints:C_0603_1608Metric
- C604: renamed from C504; footprint Capacitor_SMD:C_0805_2012Metric -> geeks-ecu-footprints:C_0805_2012Metric
- C605: renamed from C505; footprint Capacitor_SMD:C_0603_1608Metric -> geeks-ecu-footprints:C_0603_1608Metric
- C606: renamed from C506; footprint Capacitor_SMD:C_0603_1608Metric -> geeks-ecu-footprints:C_0603_1608Metric
- C607: renamed from C507; footprint Capacitor_THT:CP_Radial_D8.0mm_P3.50mm -> geeks-ecu-footprints:CP_Radial_D8.0mm_P3.50mm
- C608: footprint Capacitor_THT:CP_Radial_D8.0mm_P3.50mm -> geeks-ecu-footprints:CP_Radial_D8.0mm_P3.50mm
- NT601: renamed from NT501; footprint NetTie:NetTie-2_SMD_Pad0.5mm -> geeks-ecu-footprints:NetTie-2_SMD_Pad0.5mm
- NT602: renamed from NT502; footprint NetTie:NetTie-2_SMD_Pad0.5mm -> geeks-ecu-footprints:NetTie-2_SMD_Pad0.5mm
- Q601: renamed from Q602; footprint Package_DFN_QFN:PQFN-8-EP_6x5mm_P1.27mm_Generic -> geeks-ecu-footprints:PQFN-8-EP_6x5mm_P1.27mm_Generic
- Q602: renamed from Q603; footprint Package_DFN_QFN:PQFN-8-EP_6x5mm_P1.27mm_Generic -> geeks-ecu-footprints:PQFN-8-EP_6x5mm_P1.27mm_Generic
- Q603: renamed from Q605; footprint Package_DFN_QFN:PQFN-8-EP_6x5mm_P1.27mm_Generic -> geeks-ecu-footprints:PQFN-8-EP_6x5mm_P1.27mm_Generic
- Q604: renamed from Q601; footprint Package_DFN_QFN:PQFN-8-EP_6x5mm_P1.27mm_Generic -> geeks-ecu-footprints:PQFN-8-EP_6x5mm_P1.27mm_Generic
- R601: renamed from R501; footprint Resistor_SMD:R_0603_1608Metric -> geeks-ecu-footprints:R_0603_1608Metric
- R602: renamed from R502; footprint Resistor_SMD:R_0603_1608Metric -> geeks-ecu-footprints:R_0603_1608Metric
- R603: renamed from R503; footprint Resistor_SMD:R_0603_1608Metric -> geeks-ecu-footprints:R_0603_1608Metric
- R604: renamed from R504; footprint Resistor_SMD:R_0603_1608Metric -> geeks-ecu-footprints:R_0603_1608Metric
- R605: renamed from R505; footprint Resistor_SMD:R_2512_6332Metric -> geeks-ecu-footprints:R_2512_6332Metric
- U601: renamed from U501; footprint Package_DFN_QFN:Texas_RGE0024H_VQFN-24-1EP_4x4mm_P0.5mm_EP2.7x2.7mm -> geeks-ecu-footprints:Texas_RGE0024H_VQFN-24-1EP_4x4mm_P0.5mm_EP2.7x2.7mm
