File: hardware/Ryder/geeks-ecu/DRV8701_LowCurrent.kicad_sch (KiCad schematic)
At the start: 20 parts, among them Q801 60V 45A, Q802 60V 45A, Q803 60V 45A, Q804 60V 45A, U801 DRV8701P

Commit message: Finalize Ryder ECU
Parts:
- R802: MPN C22548 -> C21190
