File: hardware/Drive Systems/Control Panel (No Touch)/ControlPanel_CapacitiveTouch/ControlPanel_CapacitiveTouch.kicad_pcb (KiCad board)
At the start: 4 copper layers, 50.2 x 30.5 mm, 27 parts, among them J1 Conn_01x03_Pin, J2 Conn_01x03_Pin, J3 Conn_01x03_Pin, J4 Adafruit TPS61040, J5 5v Power Input, J6 Conn_01x02_Pin, J7 Conn_01x02_Pin, J8 Conn_01x02_Pin, Q1 2N7002, Q2 2N7002, Q3 2N7002

Commit message: Capacitive Touch CP v2
Parts:
- J6: value Conn_01x02_Pin -> Left; footprint Connector_JST:JST_XH_B2B-XH-A_1x02_P2.50mm_Vertical -> Connector_JST:JST_SH_BM03B-SRSS-TB_1x03-1MP_P1.00mm_Vertical
- J7: value Conn_01x02_Pin -> Center; footprint Connector_JST:JST_XH_B2B-XH-A_1x02_P2.50mm_Vertical -> Connector_JST:JST_SH_BM03B-SRSS-TB_1x03-1MP_P1.00mm_Vertical
- J8: value Conn_01x02_Pin -> Right; footprint Connector_JST:JST_XH_B2B-XH-A_1x02_P2.50mm_Vertical -> Connector_JST:JST_SH_BM03B-SRSS-TB_1x03-1MP_P1.00mm_Vertical
Connections:
- J6 pad 1: GND -> unconnected-(J6-Pin_1-Pad1)
- J7 pad 1: GND -> unconnected-(J7-Pin_1-Pad1)
- J8 pad 1: GND -> unconnected-(J8-Pin_1-Pad1)
Routing:
- net RIGHT_ACTIVE_LOW: track 12.1 -> 14.1 mm
- net LEFT_ACTIVE_LOW: track 10.5 -> 9.33 mm
- net GND: vias 28 -> 27
Other:
- board text added: "Capactive Touch 12v Adapter v2"
- board text added: "Center"
- board text added: "Left"
- board text added: "Right"
- board text removed: "Capactive Touch 12v Adapter v1"
